Commit message: added test worlds, with ramp

File: grasslammer2_description/urdf/oakd-pro-W.xacro (robot description, xacro)
@@ -30,5 +30,6 @@
       <joint name="camera_optical_joint" type="fixed">
       <!-- Point cloud frustrum is 90 degrees off from visual frame -->
-           <origin rpy="-1.57079632769 0 -1.570796332769" xyz="0 0 0" />
+           <!-- <origin rpy="-1.57079632769 0 -1.570796332769" xyz="0 0 0" /> -->
+           <origin rpy="0.0 0 0.0" xyz="0 0 0" />
 	   <parent link="oakd_${mount_point}" />
 	   <child link="camera_optical_frame" />
@@ -57,14 +58,15 @@
   </link>
   <!-- Gazebo plugin for greyscale left/right stereo pairs -->
-  <gazebo reference="oakd_${mount_point}">
+  <gazebo reference="camera_optical_frame"><!-- oakd_${mount_point}" -->
     <material>Gazebo/Grey3</material>
     <sensor type="multicamera" name="stereo_camera">
-      <update_rate>120.0</update_rate>
+      <update_rate>30.0</update_rate>
       <camera name="left">
-        <horizontal_fov>2.21</horizontal_fov> <!-- 127° -->
+        <pose>0 -0.035 0 0 0 0</pose>
+        <horizontal_fov>2.21</horizontal_fov>  <!--127°-->
         <image>
           <width>1280</width>
           <height>800</height>
-	        <format>L8</format>
+	        <format>R8G8B8</format>
         </image>
         <clip>
@@ -72,17 +74,17 @@
           <far>35</far>
         </clip>
-        <noise>
+        <!-- <noise>
           <type>gaussian</type>
           <mean>0.0</mean>
           <stddev>0.007</stddev>
-        </noise>
+        </noise> -->
       </camera>
       <camera name="right">
-        <pose>0 -0.07 0 0 0 0</pose>
+        <pose>0 0.035 0 0 0 0</pose>
         <horizontal_fov>2.21</horizontal_fov>
         <image>
           <width>1280</width>
           <height>800</height>
-	        <format>L8</format>
+	        <format>R8G8B8</format>
         </image>
         <clip>
@@ -90,15 +92,25 @@
           <far>35</far>
         </clip>
-        <noise>
+        <!-- <noise>
           <type>gaussian</type>
           <mean>0.0</mean>
           <stddev>0.007</stddev>
-        </noise>
+        </noise> -->
       </camera>
       <plugin name="stereo_camera_controller" filename="libgazebo_ros_camera.so">
-        <camera_name>stereo_camera</camera_name>
-        <frame_name>scamera_optical_frame</frame_name>
+        <camera_name></camera_name>
+        <frame_name>camera_optical_frame</frame_name>
+        <hackBaseline>0.07</hackBaseline>
+        <distortionK1>0.0</distortionK1>
+        <distortionK2>0.0</distortionK2>
+        <distortionK3>0.0</distortionK3>
+        <distortionT1>0.0</distortionT1>
+        <distortionT2>0.0</distortionT2>
         <ros>
-          <namespace>scamera</namespace>
+          <namespace></namespace>
+           <remapping>stereo_camera/left/image_raw:=/left/image_raw</remapping>
+          <remapping>stereo_camera/right/image_raw:=/right/image_raw</remapping>
+          <remapping>stereo_camera/left/camera_info:=/left/camera_info</remapping>
+          <remapping>stereo_camera/right/camera_info:=/right/camera_info</remapping>
         </ros>
       </plugin>
@@ -132,5 +144,5 @@
       <plugin name="camera_controller" filename="libgazebo_ros_camera.so">
         <camera_name>rgb_camera</camera_name>
-        <frame_name>rgb_camera_optical_frame</frame_name>
+        <frame_name>camera_rgb_optical_frame</frame_name>
         <ros>
           <namespace>rgb_camera</namespace>

File: grasslammer2_description/urdf/wheels.xacro (robot description, xacro)
@@ -36,6 +36,6 @@
             <kp>1e6</kp>
             <kd>1.0</kd>
-            <mu1>0.6</mu1>
-            <mu2>0.5</mu2>
+            <mu1>0.8</mu1>
+            <mu2>0.3</mu2>
             <fdir1 value="1 0 0"/>
             <material>Gazebo/Gray</material>
