Commit message: added tests worlds

File: grasslammer2_description/urdf/lidar.xacro (robot description, xacro)
@@ -30,5 +30,5 @@
             <pose> 0 0 0 0 0 0 </pose>
             <visualize>true</visualize>
-            <update_rate>10</update_rate>
+            <update_rate>5</update_rate>
             <ray>
                 <scan>

File: grasslammer2_description/urdf/model.urdf (robot description, URDF)
Before this commit: robot grasslammer, 4 links, 4 joints
Links:
- link base_link: geometry collision mesh filename=$(find grasslammer2_description)/meshes/rocker_body.dae; visual mesh filename=$(find grasslammer2_description)/meshes/rocker_body.dae

Commit message: fix robot model Rviz visualization

File: grasslammer2_description/urdf/lidar.xacro (robot description, xacro)
@@ -46,5 +46,5 @@
             <plugin name="laser_controller" filename="libgazebo_ros_ray_sensor.so">
                 <ros>
-                    <argument>~/out:=scan</argument>
+                    <remapping>~/out:=/scan</remapping>
                 </ros>
                 <output_type>sensor_msgs/LaserScan</output_type>

File: grasslammer2_description/urdf/model.urdf (robot description, URDF)
Before this commit: robot grasslammer, 4 links, 4 joints
Links:
- link base_link: geometry collision mesh filename=file://$(find grasslammer2_description)/meshes/rocker_body.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; visual mesh filename=file://$(find grasslammer2_description)/meshes/rocker_body.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
- link left_bar: geometry collision mesh filename=file://$(find grasslammer2_description)/meshes/rocker_L_leg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; visual mesh filename=file://$(find grasslammer2_description)/meshes/rocker_L_leg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
- link right_bar: geometry collision mesh filename=file://$(find grasslammer2_description)/meshes/rocker_R_leg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; visual mesh filename=file://$(find grasslammer2_description)/meshes/rocker_R_leg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

File: grasslammer2_description/urdf/oakd-pro-W.xacro (robot description, xacro)
@@ -13,5 +13,5 @@
               <origin rpy="0 0 0" xyz="0 0 0" />
               <geometry>
-                      <mesh filename="$(find grasslammer2_description)/meshes/OAK-D_pro.dae"/>
+                      <mesh filename="file://$(find grasslammer2_description)/meshes/OAK-D_pro.dae"/>
               </geometry>
                <material name="black" />

File: grasslammer2_description/urdf/wheels.xacro (robot description, xacro)
@@ -8,10 +8,10 @@
             <visual>
                 <geometry>
-                    <mesh filename="$(find grasslammer2_description)/meshes/rocker_wheel.stl"/>
+                    <mesh filename="file://$(find grasslammer2_description)/meshes/rocker_wheel.stl"/>
                 </geometry>
             </visual>
             <collision>
                 <geometry>
-                    <mesh filename="$(find grasslammer2_description)/meshes/rocker_wheel.stl"/>
+                    <mesh filename="file://$(find grasslammer2_description)/meshes/rocker_wheel.stl"/>
                 </geometry>
             </collision>

Commit message: now simulated velodyne is equal to the real one

File: grasslammer2_description/urdf/lidar.xacro (robot description, xacro)
@@ -34,5 +34,5 @@
                 <scan>
                     <horizontal>
-                        <samples>720</samples>
+                        <samples>2702</samples>
                         <min_angle>-2.62</min_angle>
                         <max_angle>2.62</max_angle>

File: velodyne_simulator/velodyne_description/urdf/HDL-32E.urdf.xacro (robot description, xacro)
@@ -2,5 +2,5 @@
 <robot xmlns:xacro="http://www.ros.org/wiki/xacro" name="HDL-32E">
   <xacro:property name="M_PI" value="3.1415926535897931" />
-  <xacro:macro name="HDL-32E" params="*origin parent:=base_link name:=velodyne tf_prefix:='' topic:=/velodyne_points organize_cloud:=false hz:=10 lasers:=32 samples:=2187 collision_range:=0.3 min_range:=0.9 max_range:=130.0 noise:=0.008 min_angle:=-${M_PI} max_angle:=${M_PI} gpu:=false">
+  <xacro:macro name="HDL-32E" params="*origin parent:=base_link name:=velodyne tf_prefix:='' topic:=/velodyne_points organize_cloud:=false hz:=10 lasers:=32 samples:=2185 collision_range:=0.3 min_range:=0.5 max_range:=130.0 noise:=0.008 min_angle:=-${M_PI} max_angle:=${M_PI} gpu:=false">
     <joint name="${name}_base_mount_joint" type="fixed">
       <xacro:insert_block name="origin" />
